File: Power_Systems_Complete/blue_bank.kicad_sch (KiCad schematic)
At the start: 64 parts

Commit message: completed tf and pf
Parts:
- added D? (x4): 70HFR60, symbol Device:D
- added R? (x8): 2K, symbol Device:R_US
- added R? (x4): 15, symbol Device:R_US
Connections:
- net + Charging: now also R?.1, R?.1, R?.1, R?.1
- net + Dump: now also D?.1 (K), D?.1 (K)
- net - Charging: now also R?.1, R?.1, R?.1, R?.1
- net - Dump: now also D?.2 (A), D?.2 (A)
- net Capacitor Tray/- renamed Out 1 -
- net Capacitor Tray1/+ renamed Out 1 +
- net Capacitor Tray10/- renamed Out 6 -
- net Capacitor Tray11/+ renamed Out 6 +
- net Capacitor Tray12/- renamed Out 7 -
- net Capacitor Tray13/+ renamed Out 7 +
- net Capacitor Tray14/- renamed Out 8 -
- net Capacitor Tray15/+ renamed Out 8 +
- net Capacitor Tray2/- renamed Out 2 -
- net Capacitor Tray3/+ renamed Out 2 +
- net Capacitor Tray4/- renamed Out 3 -
- net Capacitor Tray5/+ renamed Out 3 +
- net Capacitor Tray6/- renamed Out 4 -
- net Capacitor Tray7/+ renamed Out 4 +
- net Capacitor Tray8/- renamed Out 5 -
- net Capacitor Tray9/+ renamed Out 5 +
- new net: D?.1 (K), R?.1 (x2)
- new net: D?.2 (A), R?.1 (x2)
- new net Out 10 +: R?.2, R?.2, R?.2
- new net Out 10 -: R?.2, R?.2, R?.2
- new net Out 9 +: R?.2, R?.2, R?.2
- new net Out 9 -: R?.2, R?.2, R?.2
Other:
- added sheet Capacitor Tray32 (cap_tray.kicad_sch)
- added sheet Capacitor Tray33 (cap_tray.kicad_sch)
- added sheet Capacitor Tray34 (cap_tray.kicad_sch)
- added sheet Capacitor Tray35 (cap_tray.kicad_sch)

Commit message: Made changes
Changed lines of the file:
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@@
 (kicad_sch
-	(version 20231120)
+	(version 20250114)
 	(generator "eeschema")
-	(generator_version "8.0")
+	(generator_version "9.0")
 	(paper "A4" portrait)
+	(text "Dump -  and Dump + both connect to GND\nin dump configuration thru the relays"
+		(exclude_from_sim no)
+		(at 17.018 19.812 0)
+		(effects
+			(font
+				(size 1.27 1.27)
+			)
+			(justify left)
+		)
+	)
 	(junction
 		(at 111.76 154.94)
@@
 	)
 	(junction
+		(at 77.47 31.75)
+		(diameter 0)
+		(color 0 0 0 0)
+	)
+	(junction
 		(at 102.87 200.66)
 		(diameter 0)
@@
 	)
 	(junction
-		(at 77.47 30.48)
-		(diameter 0)
-		(color 0 0 0 0)
-	)
-	(junction
 		(at 130.81 163.83)
 		(diameter 0)
@@
 	(wire
 		(pts
-			(xy 81.28 19.05) (xy 81.28 30.48)
+			(xy 81.28 19.05) (xy 81.28 31.75)
 		)
 		(stroke
@@
 	(wire
 		(pts
-			(xy 77.47 29.21) (xy 77.47 30.48)
-		)
-		(stroke
-			(width 0)
-			(type default)
-		)
-	)
-	(wire
-		(pts
 			(xy 111.76 151.13) (xy 111.76 154.94)
 		)
@@
 	(wire
 		(pts
-			(xy 77.47 30.48) (xy 77.47 57.15)
-		)
-		(stroke
-			(width 0)
-			(type default)
-		)
-	)
-	(wire
-		(pts
 			(xy 49.53 191.77) (xy 50.8 191.77)
 		)
@@
 	(wire
 		(pts
+			(xy 77.47 29.21) (xy 77.47 31.75)
+		)
+		(stroke
+			(width 0)
+			(type default)
+		)
+	)
+	(wire
+		(pts
 			(xy 34.29 163.83) (xy 35.56 163.83)
 		)
@@
 	(wire
 		(pts
-			(xy 77.47 30.48) (xy 81.28 30.48)
+			(xy 77.47 31.75) (xy 81.28 31.75)
 		)
 		(stroke
@@
 	(wire
 		(pts
+			(xy 77.47 31.75) (xy 77.47 57.15)
+		)
+		(stroke
+			(width 0)
+			(type default)
+		)
+	)
+	(wire
+		(pts
 			(xy 130.81 200.66) (xy 130.81 218.44)
 		)
@@
 		)
 	)
-	(text "Dump -  and Dump + both connect to GND\nin dump configuration thru the relays"
-		(exclude_from_sim no)
-		(at 17.018 19.812 0)
-		(effects
-			(font
-				(size 1.27 1.27)
-			)
-			(justify left)
-		)
-	)
 	(hierarchical_label "Out 8 +"
 		(shape input)
 		(at 100.33 181.61 90)
-		(fields_autoplaced yes)
 		(effects
 			(font
@@
 		(shape input)
 		(at 54.61 200.66 90)
-		(fields_autoplaced yes)
 		(effects
 			(font
@@
 		(shape input)
 		(at 100.33 110.49 90)
-		(fields_autoplaced yes)
 		(effects
 			(font
@@
 		(shape input)
 		(at 54.61 92.71 90)
-		(fields_autoplaced yes)
 		(effects
 			(font
@@
 		(shape input)
 		(at 54.61 218.44 90)
-		(fields_autoplaced yes)
 		(effects
 			(font
@@
 		(shape input)
 		(at 100.33 74.93 90)
-		(fields_autoplaced yes)
 		(effects
 			(font
@@
 		(shape input)
 		(at 100.33 218.44 90)
-		(fields_autoplaced yes)
 		(effects
 			(font
@@
 		(shape input)
 		(at 100.33 200.66 90)
-		(fields_autoplaced yes)
 		(effects
 			(font
@@
 		(shape input)
 		(at 54.61 57.15 90)
-		(fields_autoplaced yes)
 		(effects
 			(font
@@
 		(shape input)
 		(at 67.31 29.21 90)
-		(fields_autoplaced yes)
 		(effects
 			(font
@@
 		(shape input)
 		(at 54.61 146.05 90)
-		(fields_autoplaced yes)
 		(effects
 			(font
@@
 		(shape input)
 		(at 54.61 181.61 90)
-		(fields_autoplaced yes)
 		(effects
 			(font
@@
 		(shape input)
 		(at 100.33 128.27 90)
-		(fields_autoplaced yes)
 		(effects
 			(font
@@
 		(shape input)
 		(at 77.47 29.21 90)
-		(fields_autoplaced yes)
 		(effects
 			(font
@@
 		(shape input)
 		(at 54.61 74.93 90)
-		(fields_autoplaced yes)
 		(effects
 			(font
@@
 		(shape input)
 		(at 100.33 92.71 90)
-		(fields_autoplaced yes)
 		(effects
 			(font
@@
 		(shape input)
 		(at 54.61 110.49 90)
-		(fields_autoplaced yes)
 		(effects
 			(font
@@
 		(shape input)
 		(at 100.33 146.05 90)
-		(fields_autoplaced yes)
 		(effects
 			(font
@@
 		(shape input)
 		(at 88.9 29.21 90)
-		(fields_autoplaced yes)
 		(effects
 			(font
@@
 		(shape input)
 		(at 83.82 29.21 90)
-		(fields_autoplaced yes)
 		(effects
 			(font
@@
 		(shape input)
 		(at 54.61 163.83 90)
-		(fields_autoplaced yes)
 		(effects
 			(font
@@
 		(shape input)
 		(at 100.33 57.15 90)
-		(fields_autoplaced yes)
 		(effects
 			(font
@@
 		(shape input)
 		(at 71.12 29.21 90)
-		(fields_autoplaced yes)
 		(effects
 			(font
@@
 		(shape input)
 		(at 100.33 163.83 90)
-		(fields_autoplaced yes)
 		(effects
 			(font
@@
 		(shape input)
 		(at 54.61 128.27 90)
-		(fields_autoplaced yes)
 		(effects
 			(font
@@
 					(unit 1)
 				)
+				(path "/c716675b-d754-4b87-99eb-660dfcc257fb/b111d471-3bf5-464d-8502-0d5689b200c0"
+					(reference "D?")
+					(unit 1)
+				)
 				(path "/c716675b-d754-4b87-99eb-660dfcc257fb/b3e11a39-5b02-4e5b-bb09-92d8c9f1dda7"
 					(reference "D?")
@@
 		(at 83.82 90.17)
 		(size 12.7 5.08)
+		(exclude_from_sim no)
+		(in_bom yes)
+		(on_board yes)
+		(dnp no)
 		(fields_autoplaced yes)
 		(stroke
@@
 		(at 57.15 90.17)
 		(size 12.7 5.08)
+		(exclude_from_sim no)
+		(in_bom yes)
+		(on_board yes)
+		(dnp no)
 		(fields_autoplaced yes)
 		(stroke
@@
 		(at 83.82 161.29)
 		(size 12.7 5.08)
+		(exclude_from_sim no)
+		(in_bom yes)
+		(on_board yes)
+		(dnp no)
 		(fields_autoplaced yes)
 		(stroke
@@
 		(at 83.82 107.95)
 		(size 12.7 5.08)
+		(exclude_from_sim no)
+		(in_bom yes)
+		(on_board yes)
+		(dnp no)
 		(fields_autoplaced yes)
 		(stroke
@@
 		(at 57.15 54.61)
 		(size 12.7 5.08)
+		(exclude_from_sim no)
+		(in_bom yes)
+		(on_board yes)
+		(dnp no)
 		(fields_autoplaced yes)
 		(stroke
@@
 		(at 57.15 125.73)
 		(size 12.7 5.08)
+		(exclude_from_sim no)
+		(in_bom yes)
+		(on_board yes)
+		(dnp no)
 		(fields_autoplaced yes)
 		(stroke
@@
 		(at 83.82 125.73)
 		(size 12.7 5.08)
+		(exclude_from_sim no)
+		(in_bom yes)
+		(on_board yes)
+		(dnp no)
 		(fields_autoplaced yes)
 		(stroke
@@
 		(at 57.15 215.9)
 		(size 12.7 5.08)
+		(exclude_from_sim no)
+		(in_bom yes)
+		(on_board yes)
+		(dnp no)
 		(fields_autoplaced yes)
 		(stroke
@@
 		(at 83.82 72.39)
 		(size 12.7 5.08)
+		(exclude_from_sim no)
+		(in_bom yes)
+		(on_board yes)
+		(dnp no)
 		(fields_autoplaced yes)
 		(stroke
@@
 		(at 57.15 179.07)
 		(size 12.7 5.08)
+		(exclude_from_sim no)
+		(in_bom yes)
+		(on_board yes)
+		(dnp no)
 		(fields_autoplaced yes)
 		(stroke
@@
 		(at 83.82 54.61)
 		(size 12.7 5.08)
+		(exclude_from_sim no)
+		(in_bom yes)
+		(on_board yes)
+		(dnp no)
 		(fields_autoplaced yes)
 		(stroke
@@
 		(at 83.82 215.9)
 		(size 12.7 5.08)
+		(exclude_from_sim no)
+		(in_bom yes)
+		(on_board yes)
+		(dnp no)
 		(fields_autoplaced yes)
 		(stroke
@@
 		(at 57.15 107.95)
 		(size 12.7 5.08)
+		(exclude_from_sim no)
+		(in_bom yes)
+		(on_board yes)
+		(dnp no)
 		(fields_autoplaced yes)
 		(stroke
@@
 		(at 57.15 161.29)
 		(size 12.7 5.08)
+		(exclude_from_sim no)
+		(in_bom yes)
+		(on_board yes)
+		(dnp no)
 		(fields_autoplaced yes)
 		(stroke
@@
 		(at 57.15 143.51)
 		(size 12.7 5.08)
+		(exclude_from_sim no)
+		(in_bom yes)
+		(on_board yes)
+		(dnp no)
 		(fields_autoplaced yes)
 		(stroke
@@
 		(at 83.82 198.12)
 		(size 12.7 5.08)
+		(exclude_from_sim no)
+		(in_bom yes)
+		(on_board yes)
+		(dnp no)
 		(fields_autoplaced yes)
 		(stroke
@@
 		(at 57.15 72.39)
 		(size 12.7 5.08)
+		(exclude_from_sim no)
+		(in_bom yes)
+		(on_board yes)
+		(dnp no)
 		(fields_autoplaced yes)
 		(stroke
@@
 		(at 57.15 198.12)
 		(size 12.7 5.08)
+		(exclude_from_sim no)
+		(in_bom yes)
+		(on_board yes)
+		(dnp no)
 		(fields_autoplaced yes)
 		(stroke
@@
 		(at 83.82 179.07)
 		(size 12.7 5.08)
+		(exclude_from_sim no)
+		(in_bom yes)
+		(on_board yes)
+		(dnp no)
 		(fields_autoplaced yes)
 		(stroke
@@
 		(at 83.82 143.51)
 		(size 12.7 5.08)
+		(exclude_from_sim no)
+		(in_bom yes)
+		(on_board yes)
+		(dnp no)
 		(fields_autoplaced yes)
 		(stroke
