File: Power_Systems_Complete/CapColumn15.kicad_sch (KiCad schematic)
At the start: 15 parts

Commit message: Actual correct kicad and spice sim of red bank 1
Parts:
- renumbered C167 to C152, C168 to C153, C169 to C154, C170 to C155, C171 to C156, C172 to C157, C173 to C158, C174 to C159, C175 to C160, C176 to C161, C177 to C162, C178 to C163, C179 to C164, C180 to C165, C181 to C166
