File: Power_Systems_Complete/red_cap_bank_1.kicad_sch (KiCad schematic)
At the start: 88 parts

Commit message: Actual correct kicad and spice sim of red bank 1
Parts:
- R25, R34, R39, R40, R49, R50, R59, R60: value 2k -> 15
- R29, R30, R35, R44, R45, R54, R55, R64: value 15 -> 2k
Connections:
- net CapColumn15_2/Minus is gone; now on net CapColumn15_1/Plus: D9.2 (A)
- net CapColumn15_1/Plus: now also R26.2, R27.2; no longer D11.1 (K)
- net CapColumn15_3/Plus: now also D14.2 (A), R37.2, R38.2; no longer D13.1 (K)
- net CapColumn15_5/Plus: now also D18.2 (A), R47.2, R48.2; no longer D17.1 (K)
- net CapColumn15_7/Plus: now also D22.2 (A), R57.2, R58.2; no longer D21.1 (K)
- net MinusCharge: now also R30.2, R32.1, R42.1, R44.2, R52.1, R54.2, R62.1, R64.2; no longer R32.2, R34.1, R40.1, R42.2, R50.1, R52.2, R60.1, R62.2
- net MinusDump: now also R34.2, R40.2, R50.2, R60.2; no longer R30.2, R44.2, R54.2, R64.2
- net PlusCharge: now also R26.1, R28.2, R29.2, R35.2, R37.1, R45.2, R47.1, R55.2, R57.1; no longer R25.2, R26.2, R28.1, R37.2, R39.1, R47.2, R49.1, R57.2, R59.1
- net PlusDump: now also R25.2, R39.2, R49.2, R59.2; no longer R29.2, R35.2, R45.2, R55.2
- net at D16.1 (K), R43.1, R44.1: no longer D15.1 (K), R42.1
- net at D20.1 (K), R53.1, R54.1: no longer D19.1 (K), R52.1
- net at D24.1 (K), R63.1, R64.1: no longer D23.1 (K), R62.1
- net at D21.2 (A), R55.1, R56.1: no longer D22.2 (A), R57.1
- net at D13.2 (A), R35.1, R36.1: no longer D14.2 (A), R37.1
- net at D17.2 (A), R45.1, R46.1: no longer D18.2 (A), R47.1
- net CapColumn15_4/Minus: no longer names the net of D16.2 (A)
- net CapColumn15_4/Minus: now also D15.2 (A), R40.1
- net CapColumn15_6/Minus: no longer names the net of D20.2 (A)
- net CapColumn15_6/Minus: now also D19.2 (A), R50.1
- net CapColumn15_8/Minus: no longer names the net of D24.2 (A)
- net CapColumn15_8/Minus: now also D23.2 (A), R60.1
- new net: D13.1 (K), D14.1 (K), R39.1
- new net: D10.2 (A), R28.1, R29.1
- new net: D17.1 (K), D18.1 (K), R49.1
- new net: D11.1 (K), R30.1, R31.1
- new net: D11.2 (A), D12.2 (A), R34.1
- new net: D10.1 (K), D9.1 (K), R25.1
- new net: D21.1 (K), D22.1 (K), R59.1
- new net CapColumn15_2/Plus: D12.1 (K), R32.2, R33.2
- new net CapColumn15_4/Plus: D15.1 (K), R41.2, R42.2
- new net CapColumn15_6/Plus: D19.1 (K), R51.2, R52.2
- new net CapColumn15_8/Plus: D23.1 (K), R61.2, R62.2
